File: Proyecto/PCB/PCB.kicad_pcb (KiCad board)
At the start: 2 copper layers, 200 x 100 mm, 21 parts, among them J1 STM_L, J10 XL6009_IN+, J11 XL6009_IN-, J12 XL6009_OUT+, J13 XL6009_OUT-, J14 MAX30102, J15 PILA+, J16 PILA-, J2 STM_R, J3 Display, J4 AD620_IN, J5 AD620_OUT, J6 TP4056_OUT+, J7 TP4056_OUT-, J8 TP4056+, J9 TP4056-

Commit message: Proyecto
Parts:
- added J17: 3.3V, TestPoint:TestPoint_Pad_D2.0mm, B.Cu at (66.0, 91.0)
- added J18: 3.3V, TestPoint:TestPoint_Pad_D2.0mm, B.Cu at (134.1, 83.5)
Connections:
- J1 pad 15: unconnected-(J1-Pin_15-Pad15) -> Net-(J1-Pin_15)
- J3 pad 8: unconnected-(J3-Pin_8-Pad8) -> Net-(J17-Pin_1)
Routing:
- net Net-(J17-Pin_1): track 0.00 -> 7.88 mm
- net Net-(J1-Pin_15): track 0.00 -> 6.28 mm

Commit message: Proyecto TD2
Parts:
- removed J14: MAX30102, Connector_Wire:SolderWire-0.5sqmm_1x05_P4.6mm_D0.9mm_OD2.1mm
- added J19: Display_2, Connector_PinSocket_2.54mm:PinSocket_1x05_P2.54mm_Vertical, F.Cu at (67.9, 55.5)
- added J20: MAX30102_2, Connector_PinSocket_2.54mm:PinSocket_1x01_P2.54mm_Vertical, F.Cu at (75.5, 144.2)
- added J21: MAX30102_3, Connector_PinSocket_2.54mm:PinSocket_1x01_P2.54mm_Vertical, F.Cu at (75.5, 128.9)
- added J22: MAX30102_1, Connector_PinSocket_2.54mm:PinSocket_1x07_P2.54mm_Vertical, F.Cu at (86.5, 144.2)
- J3: value Display -> Display_1
- moved J8 157.6 mm to (114.0, 58.0), turned to -90 degrees
- moved J9 143.9 mm to (114.0, 72.0), turned to -90 degrees
- moved C2 131.0 mm to (62.8, 126.0)
- moved J16 127.5 mm to (105.0, 69.5), turned to -90 degrees
- moved J15 127.1 mm to (105.0, 60.5), turned to -90 degrees
- moved J6 123.4 mm to (136.0, 58.0), turned to 0 degrees
- moved C3 116.1 mm to (70.5, 144.0), turned to 180 degrees
- moved J7 105.4 mm to (136.0, 72.0), turned to 180 degrees
- moved C1 98.3 mm to (180.2, 145.0), turned to 0 degrees
- moved J10 91.1 mm to (153.0, 59.0), turned to 90 degrees
- moved J11 88.0 mm to (153.0, 72.0), turned to 90 degrees
- moved J1 62.8 mm to (164.4, 138.7), turned to 180 degrees
- moved J4 51.7 mm to (180.2, 134.5)
- moved J5 51.7 mm to (180.2, 106.5)
- moved J2 49.0 mm to (102.9, 138.7), turned to 180 degrees
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Connections:
- J2 pad 10: GND -> unconnected-(J2-Pin_10-Pad10)
Routing:
- net /D_SD/MOSI: track 148.4 -> 41.5 mm
- net /D_SDO/MISO: track 122.5 -> 28.9 mm
- net /D_SCK: track 110.9 -> 36.4 mm
- net /Salida_AD620: track 98.9 -> 32.6 mm
- net /D_DC/RS: track 97.1 -> 47.3 mm
- net /Vcc: track 219.8 -> 266.1 mm
- net /D_CS: track 88.6 -> 109.5 mm
- net /PILA+: track 50.2 -> 31.0 mm
- net /TP4056_OUT+: track 30.6 -> 17.4 mm
- net /S_INT: track 37.2 -> 29.9 mm
- net /PILA-: track 24.3 -> 31.0 mm
- net /S_SDA: track 39.0 -> 35.0 mm
- net Net-(J17-Pin_1): track 7.88 -> 5.34 mm
- net Net-(J1-Pin_15): track 6.28 -> 7.95 mm
- net /S_SCL: track 64.4 -> 62.8 mm
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Other:
- board size 200 x 100 mm -> 150 x 100 mm

Commit message: Proyecto V2
Parts:
- removed J15: PILA+, Connector_PinSocket_2.54mm:PinSocket_1x01_P2.54mm_Vertical
- removed J16: PILA-, Connector_PinSocket_2.54mm:PinSocket_1x01_P2.54mm_Vertical
- added J14: Conn_01x02_Pin, TerminalBlock_Phoenix:TerminalBlock_Phoenix_MKDS-1,5-2-5.08_1x02_P5.08mm_Horizontal, F.Cu at (112.5, 56.0)
- added SW1: SW_SPDT, Button_Switch_THT:SW_Slide_SPDT_Straight_CK_OS102011MS2Q, F.Cu at (147.0, 55.5)
- moved J6 10.5 mm to (145.0, 63.3)
- moved J8 10.2 mm to (123.0, 62.8)
- moved J9 10.2 mm to (123.0, 76.8)
- moved J7 10.0 mm to (145.0, 76.4)
- moved J11 5.60 mm to (156.5, 76.4)
- moved J13 5.60 mm to (196.5, 76.4)
- moved J10 3.50 mm to (156.5, 58.9)
- moved J12 3.50 mm to (196.5, 58.9)
- moved D1 3.00 mm to (160.0, 84.5)
- moved R1 3.00 mm to (175.1, 84.5)
- moved J17 2.51 mm to (80.7, 113.5)
- moved J3 2.51 mm to (62.9, 118.8)
- moved J19 0.58 mm to (68.2, 55.0)
- moved J5 0.50 mm to (180.2, 106.0)
Connections:
- J10 pad 1: /TP4056_OUT+ -> Net-(J10-Pin_1)
Routing:
- net /PILA-: track 31.0 -> 53.5 mm
- net Net-(J10-Pin_1): track 0.00 -> 12.1 mm
- net /D_CS: track 109.5 -> 97.5 mm
- net /PILA+: track 31.0 -> 41.3 mm
- net /TP4056_OUT+: track 17.4 -> 7.81 mm
- net /D_RESET: track 85.7 -> 77.7 mm
- net /Vcc: track 266.1 -> 260.6 mm
- net /TP4056_OUT-: track 17.0 -> 11.6 mm
- net /AD620_Vout: track 34.3 -> 30.7 mm
- net /D_SCK: track 36.4 -> 39.7 mm
- net /D_SDO/MISO: track 28.9 -> 32.2 mm
- net /Salida_AD620: track 32.6 -> 29.6 mm
- net /D_SD/MOSI: track 41.5 -> 44.4 mm
- net /D_DC/RS: track 47.3 -> 49.9 mm

Commit message: Proyecto V2
Other:
- board text added: "UTN FRBA PROYECTO TD2 R4001"
Changed lines of the file:
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@@
 			(crossoutdnponfab yes)
 			(subtractmaskfromsilk no)
-			(outputformat 5)
+			(outputformat 4)
 			(mirror no)
 			(drillshape 1)
@@
 		(layer "Edge.Cuts")
 	)
-	(segment
-		(start 109.21 69.46)
-		(end 107.42 67.67)
-		(width 1.5)
-		(layer "B.Cu")
-		(net "/PILA-")
-	)
-	(segment
-		(start 107.42 67.67)
-		(end 107.42 56)
-		(width 1.5)
-		(layer "B.Cu")
-		(net "/PILA-")
-	)
-	(segment
-		(start 145 71)
-		(end 143.46 69.46)
-		(width 1.5)
-		(layer "B.Cu")
-		(net "/PILA-")
-	)
-	(segment
-		(start 145 73.71)
-		(end 145 71)
-		(width 1.5)
-		(layer "B.Cu")
-		(net "/PILA-")
-	)
-	(segment
-		(start 144.88 73.83)
-		(end 145 73.71)
-		(width 1.5)
-		(layer "B.Cu")
-		(net "/PILA-")
-	)
-	(segment
-		(start 143.46 69.46)
-		(end 109.21 69.46)
-		(width 1.5)
+	(gr_text "UTN FRBA\nPROYECTO TD2\nR4001\n"
+		(at 141 108.5 0)
 		(layer "B.Cu")
-		(net "/PILA-")
+		(effects
+			(font
+				(size 1.5 1.5)
+				(thickness 0.3)
+				(bold yes)
+			)
+			(justify left bottom mirror)
+		)
 	)
 	(segment
@@
 	)
 	(segment
+		(start 109.21 69.46)
+		(end 107.42 67.67)
+		(width 1.5)
+		(layer "B.Cu")
+		(net "/PILA-")
+	)
+	(segment
+		(start 107.42 67.67)
+		(end 107.42 56)
+		(width 1.5)
+		(layer "B.Cu")
+		(net "/PILA-")
+	)
+	(segment
+		(start 145 71)
+		(end 143.46 69.46)
+		(width 1.5)
+		(layer "B.Cu")
+		(net "/PILA-")
+	)
+	(segment
+		(start 145 73.71)
+		(end 145 71)
+		(width 1.5)
+		(layer "B.Cu")
+		(net "/PILA-")
+	)
+	(segment
+		(start 144.88 73.83)
+		(end 145 73.71)
+		(width 1.5)
+		(layer "B.Cu")
+		(net "/PILA-")
+	)
+	(segment
+		(start 143.46 69.46)
+		(end 109.21 69.46)
+		(width 1.5)
+		(layer "B.Cu")
+		(net "/PILA-")
+	)
+	(segment
+		(start 147 55.5)
+		(end 147 57.5)
+		(width 1.5)
+		(layer "B.Cu")
+		(net "Net-(J10-Pin_1)")
+	)
+	(segment
+		(start 147 57.5)
+		(end 148.37 58.87)
+		(width 1.5)
+		(layer "B.Cu")
+		(net "Net-(J10-Pin_1)")
+	)
+	(segment
+		(start 148.37 58.87)
+		(end 156.5 58.87)
+		(width 1.5)
+		(layer "B.Cu")
+		(net "Net-(J10-Pin_1)")
+	)
+	(segment
+		(start 145 55.5)
+		(end 145 63.31)
+		(width 1.5)
+		(layer "B.Cu")
+		(net "/TP4056_OUT+")
+	)
+	(segment
 		(start 175.08 84.5)
 		(end 183.5 84.5)
@@
 	)
 	(segment
-		(start 145 55.5)
-		(end 145 63.31)
-		(width 1.5)
-		(layer "B.Cu")
-		(net "/TP4056_OUT+")
-	)
-	(segment
 		(start 69.25 86)
 		(end 110.5 86)
@@
 		(net "/PILA+")
 	)
-	(segment
-		(start 147 55.5)
-		(end 147 57.5)
-		(width 1.5)
-		(layer "B.Cu")
-		(net "Net-(J10-Pin_1)")
-	)
-	(segment
-		(start 147 57.5)
-		(end 148.37 58.87)
-		(width 1.5)
-		(layer "B.Cu")
-		(net "Net-(J10-Pin_1)")
-	)
-	(segment
-		(start 148.37 58.87)
-		(end 156.5 58.87)
-		(width 1.5)
-		(layer "B.Cu")
-		(net "Net-(J10-Pin_1)")
-	)
 	(zone

Commit message: Proyecto V2
Parts:
- added J15: Bornera_Electrodo, TerminalBlock_Phoenix:TerminalBlock_Phoenix_MKDS-1,5-2-5.08_1x02_P5.08mm_Horizontal, F.Cu at (193.7, 145.3)
- J14: value Conn_01x02_Pin -> Bornera_Pila
- moved C1 3.51 mm to (180.5, 141.5), turned to 180 degrees
- moved J4 2.02 mm to (180.5, 132.5)
- moved J5 2.02 mm to (180.5, 104.0)
Connections:
- J4 pad 3: unconnected-(J4-Pin_3-Pad3) -> /S-
- J4 pad 4: unconnected-(J4-Pin_4-Pad4) -> /S+
Routing:
- net /S-: track 0.00 -> 20.0 mm
- net /S+: track 0.00 -> 12.3 mm
- net /AD620_Vout: track 30.7 -> 28.8 mm

Commit message: Proyecto V2
Routing:
- net /D_RESET: track 77.7 -> 79.1 mm
Changed lines of the file:
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@@
 			(crossoutdnponfab yes)
 			(subtractmaskfromsilk no)
-			(outputformat 5)
+			(outputformat 4)
 			(mirror no)
 			(drillshape 1)
@@
 	)
 	(segment
-		(start 107.5 89.5)
-		(end 109 91)
-		(width 1)
-		(layer "B.Cu")
-		(net "/D_RESET")
-	)
-	(segment
-		(start 71.875 89.5)
-		(end 107.5 89.5)
+		(start 109 89.75)
+		(end 109 97)
 		(width 1)
 		(layer "B.Cu")
@@
 	)
 	(segment
-		(start 109 91)
-		(end 109 97)
+		(start 70.54 90.835)
+		(end 72.625 88.75)
 		(width 1)
 		(layer "B.Cu")
@@
 	)
 	(segment
-		(start 70.54 90.835)
-		(end 71.875 89.5)
+		(start 109 97)
+		(end 107.906179 98.093821)
 		(width 1)
 		(layer "B.Cu")
@@
 	)
 	(segment
-		(start 70.54 118.83)
-		(end 70.5 118.79)
-		(width 1.5)
+		(start 72.625 88.75)
+		(end 108 88.75)
+		(width 1)
 		(layer "B.Cu")
 		(net "/D_RESET")
 	)
 	(segment
-		(start 109 97)
-		(end 107.906179 98.093821)
+		(start 108 88.75)
+		(end 109 89.75)
 		(width 1)
 		(layer "B.Cu")
 		(net "/D_RESET")
+	)
+	(segment
+		(start 70.54 118.83)
+		(end 70.5 118.79)
+		(width 1.5)
+		(layer "B.Cu")
+		(net "/D_RESET")

Commit message: Proyecto V2
Parts:
- J1: value STM_L -> Conn_02x20_Odd_Even; footprint Connector_PinSocket_2.54mm:PinSocket_2x19_P2.54mm_Vertical -> Connector_PinSocket_2.54mm:PinSocket_2x20_P2.54mm_Vertical
- J2: value STM_R -> Conn_02x20_Odd_Even; footprint Connector_PinSocket_2.54mm:PinSocket_2x19_P2.54mm_Vertical -> Connector_PinSocket_2.54mm:PinSocket_2x20_P2.54mm_Vertical
- SW1: footprint Button_Switch_THT:SW_Slide_SPDT_Straight_CK_OS102011MS2Q -> Button_Switch_THT:SW_Slide-03_Wuerth-WS-SLTV_10x2.5x6.4_P2.54mm
- moved J7 24.5 mm to (120.5, 76.0), turned to 90 degrees
- moved J9 23.0 mm to (120.0, 54.0), turned to 180 degrees
- moved J6 17.1 mm to (133.5, 76.0), turned to -90 degrees
- moved J8 14.1 mm to (134.0, 54.0), turned to 180 degrees
- moved SW1 4.27 mm to (144.5, 59.0), turned to 90 degrees
- moved J14 4.03 mm to (108.5, 56.5)
- moved J10 2.00 mm to (154.5, 59.0)
- moved J12 2.00 mm to (194.5, 59.0)
- moved J11 2.00 mm to (154.5, 76.5)
- moved J13 2.00 mm to (194.5, 76.5)
- moved J2 0.29 mm to (103.0, 139.0)
- moved J1 0.27 mm to (164.5, 139.0)
Routing:
- net /TP4056_OUT-: track 11.6 -> 41.8 mm
- net /PILA-: track 53.5 -> 36.4 mm
- net /TP4056_OUT+: track 7.81 -> 24.3 mm
- net /D_CS: track 97.5 -> 101.0 mm
- net /D_RESET: track 79.1 -> 81.6 mm
- net /Vcc: track 260.6 -> 258.5 mm
- net Net-(J10-Pin_1): track 12.1 -> 10.0 mm
- net /PILA+: track 41.3 -> 39.6 mm
